File: HW/Cockpit management.sch (KiCad schematic (older format))
At the start: 26 parts, among them Q1 Q_NMOS_GSD, Q14 Q_NMOS_GSD, Q15 Q_NMOS_GSD, Q2 Q_NMOS_GSD, Q3 Q_NMOS_GSD, Q4 Q_NMOS_GSD, Q5 Q_NMOS_GSD, Q6 Q_NMOS_GSD, Q7 Q_NMOS_GSD, Q8 Q_NMOS_GSD

Commit message: Version 1.1
Version 1.1
Hw and Sw improvements
Parts:
- added R11, R4, R5: 3k, Resistor_SMD:R_0603_1608Metric_Pad1.05x0.95mm_HandSolder, symbol Device:R
- C18, C32: footprint Capacitors_SMD:C_0805 -> Capacitor_SMD:C_0805_2012Metric_Pad1.15x1.40mm_HandSolder
- Q1, Q14, Q15, Q2, Q3, Q4, Q5, Q6, Q7, Q8: footprint TO_SOT_Packages_SMD:SOT-323_SC-70 -> Package_TO_SOT_SMD:SOT-23
- R10, R36, R37, R38, R40, R41, R42, R6, R7, R8, R9: footprint Resistors_SMD:R_0603 -> Resistor_SMD:R_0603_1608Metric_Pad1.05x0.95mm_HandSolder
- R16, R17, R18: value 100k -> 33k; footprint Resistors_SMD:R_0603 -> Resistor_SMD:R_0603_1608Metric_Pad1.05x0.95mm_HandSolder
Connections:
- net BP_FAN_AUTO: now also R5.1
- net PUMP_AUTO: now also R4.1
- net RAD_FAN_AUTO: now also R11.1
- net BP_FAN_CMD renamed PWM2
- net PUMP_CMD renamed PWM3
- net RAD_FAN_CMD renamed PWM1
- new net +5V: R11.2, R4.2, R5.2
Other:
- moved on the sheet: Q7, Q8, R17, R18
