File: HW/MCU.sch (KiCad schematic (older format))
At the start: 50 parts, among them J1 Conn_02x05_Top_Bottom, Q10 Q_NMOS_GSD, Q11 Q_NMOS_GSD, Q12 BC857BDW1, Q13 Q_PMOS_GSD, Q9 Q_NMOS_GSD, SW1 SW_Push_Dual, U1 STM32F303VCTx, U2 SN65HVD234, U4 24AA02-OT

Commit message: Version 1.1
Version 1.1
Hw and Sw improvements
Parts:
- removed FL1: ACT45B-220-2P-TL003, footprint:ACT45B, symbol Dash-rescue:ACT45B-220-2P-TL003-ACT45B-220-2P-TL003
- removed Q12: BC857BDW1, TO_SOT_Packages_SMD:SOT-363_SC-70-6, symbol Transistor_BJT:BC857BDW1
- removed Q13: Q_PMOS_GSD, TO_SOT_Packages_SMD:SOT-323_SC-70, symbol Device:Q_PMOS_GSD
- removed R11, R13, R15, R4, R5: 22, Resistors_SMD:R_0603, symbol Device:R_US
- removed R25, R28: 68.1k, Resistors_SMD:R_0603, symbol Device:R_US
- removed SW1: SW_Push_Dual, footprint:pulsante, symbol Switch:SW_Push_Dual
- added C7, C8: 10p, Capacitor_SMD:C_0603_1608Metric_Pad1.05x0.95mm_HandSolder, symbol Device:C
- added L2: L_Core_Ferrite_Coupled, footprint:ACT45B, symbol Dash-rescue:L_Core_Ferrite_Coupled-Device
- added Y1: Crystal_GND24, footprint:Crystal_SMD_Abracon_ABM3B-4Pin_5.0x3.2mm, symbol Device:Crystal_GND24
- C1, C16, C17, C2, C20, C24, C25, C26, C27, C28, C29, C3, C30, C31, C4: footprint Capacitors_SMD:C_0805 -> Capacitor_SMD:C_0805_2012Metric_Pad1.15x1.40mm_HandSolder
- L1: footprint Inductors_SMD:L_0603 -> Inductor_SMD:L_0603_1608Metric_Pad1.05x0.95mm_HandSolder
- Q10, Q11, Q9: footprint TO_SOT_Packages_SMD:SOT-323_SC-70 -> Package_TO_SOT_SMD:SOT-23
- R1, R23, R24, R26, R27, R3: footprint Resistors_SMD:R_0603 -> Resistor_SMD:R_0603_1608Metric_Pad1.05x0.95mm_HandSolder
- R12: value 22 -> 0; footprint Resistors_SMD:R_0603 -> Resistor_SMD:R_0603_1608Metric_Pad1.05x0.95mm_HandSolder
- R14, R39: value 2k -> 3k; footprint Resistors_SMD:R_0603 -> Resistor_SMD:R_0603_1608Metric_Pad1.05x0.95mm_HandSolder
- R19, R20, R22: value 100k -> 33k; footprint Resistors_SMD:R_0603 -> Resistor_SMD:R_0603_1608Metric_Pad1.05x0.95mm_HandSolder
- R2: value 15k -> 33k; footprint Resistors_SMD:R_0603 -> Resistor_SMD:R_0603_1608Metric_Pad1.05x0.95mm_HandSolder
- R21: value 1.6k -> 1.2k; footprint Resistors_SMD:R_0603 -> Resistor_SMD:R_0603_1608Metric_Pad1.05x0.95mm_HandSolder
- U1: footprint Housings_QFP:LQFP-100_14x14mm_Pitch0.5mm -> Package_QFP:LQFP-100_14x14mm_P0.5mm
- U2: footprint Housings_SOIC:SOIC-8_3.9x4.9mm_Pitch1.27mm -> Package_SO:SOIC-8_3.9x4.9mm_P1.27mm
- U4: footprint TO_SOT_Packages_SMD:SOT-23-5 -> Package_TO_SOT_SMD:SOT-23-5_HandSoldering
- Z1: footprint TO_SOT_Packages_SMD:SOT-23 -> Package_TO_SOT_SMD:SOT-23
Connections:
- net +3.3v_EXT is gone; now on net +3V3: J1.10 (Pin_10), J1.6 (Pin_6)
- net BMS_Led_Cmd: now also U1.96 (PB9); no longer U1.41 (PE10)
- net Buzzer: now also U1.1 (PE2); no longer U1.25 (PA2)
- net CAN_H: now also C30.2, R26.1, Z1.2, L2.4; no longer C29.1, R27.1, Z1.1
- net CAN_L: now also C29.1, R27.1, Z1.1, L2.3; no longer C30.2, R26.1, Z1.2
- net GND: now also C7.2, C8.2, Y1.2, Y1.4
- net Imd_Err_Led_Cmd: now also U1.11 (PF10); no longer U1.45 (PE14)
- net JTDI: now also J1.2 (Pin_2)
- net No_Hv_Led: now also U1.2 (PE3); no longer U1.43 (PE12)
- net RTD_Button: now also U1.25 (PA2); no longer U1.15 (PC0)
- net Rtd_Led: now also U1.4 (PE5); no longer U1.47 (PB10)
- net SWCLK: now also J1.1 (Pin_1)
- net SWDIO: now also J1.4 (Pin_4); no longer R12.2
- net SWO: now also J1.3 (Pin_3)
- net USART_RX: now also J1.5 (Pin_5)
- net USART_TX: now also J1.7 (Pin_7)
- net gpio_BLUE: now also U1.26 (PA3); no longer U1.13 (PF1)
- net gpio_GREEN: now also U1.43 (PE12); no longer U1.3 (PE4)
- net gpio_RED: now also U1.42 (PE11); no longer U1.1 (PE2)
- net spare_button: now also U1.24 (PA1); no longer U1.17 (PC2)
- net at U1.12 (PF0): now also C7.1, Y1.1
- net at U2.6 (CANL): now also L2.2
- net at U2.7 (CANH): now also L2.1
- net at R12.1: now also U1.13 (PF1); no longer J1.4 (Pin_4)
- net Fan_Bp_Cmd renamed PWM3
- net Fan_Rad_Cmd renamed PWM2
- net Pump_Cmd renamed PWM1
- new net: C8.1, R12.2, Y1.3
Other:
- moved on the sheet: C29, C30, R26, R27
