File: HW/Power Supply.sch (KiCad schematic (older format))
At the start: 21 parts, among them U3 LM1117-3.3, U5 LMZ14202TZE-ADJ_NOPB

Commit message: Version 1.1
Version 1.1
Hw and Sw improvements
Parts:
- C15, C19, C21, C22, C33, C5: footprint Capacitors_SMD:C_0805 -> Capacitor_SMD:C_0805_2012Metric_Pad1.15x1.40mm_HandSolder
- C23: footprint Capacitors_SMD:C_1210 -> Capacitor_SMD:C_1206_3216Metric_Pad1.42x1.75mm_HandSolder
- C34: footprint Capacitors_SMD:C_0805 -> Capacitor_SMD:C_1206_3216Metric_Pad1.42x1.75mm_HandSolder
- C6: footprint Capacitors_SMD:C_1206 -> Capacitor_SMD:C_1206_3216Metric_Pad1.42x1.75mm_HandSolder
- D1: footprint Diodes_SMD:D_SOD-123 -> Diode_SMD:D_SOD-123
- D2, D3: footprint Diodes_SMD:D_0805 -> LED_SMD:LED_0805_2012Metric_Pad1.15x1.40mm_HandSolder
- R29: value 68.1k -> 68k; footprint Resistors_SMD:R_0603 -> Resistor_SMD:R_0603_1608Metric_Pad1.05x0.95mm_HandSolder
- R30, R31, R32, R33, R34, R35: footprint Resistors_SMD:R_0603 -> Resistor_SMD:R_0603_1608Metric_Pad1.05x0.95mm_HandSolder
- U3: footprint TO_SOT_Packages_SMD:SOT-223 -> Package_TO_SOT_SMD:SOT-223
Connections:
- net +5v renamed +5V
Changed lines of the file:
@@
 EESchema Schematic File Version 4
 LIBS:Dash-cache
-EELAYER 26 0
+EELAYER 29 0
 EELAYER END
 $Descr A4 11693 8268
 encoding utf-8
-Sheet 4 4
+Sheet 3 4
 Title ""
 Date ""
@@
 F 3 "http://uk.rs-online.com/web/p/products/7981195P" H 4800 1800 50  0001 L CNN
 F 4 "Voltage Regulators - Switching Regulators 2A pwr Module w/ 42V Max Input Vtg" H 4800 1700 50  0001 L CNN "Description"
-F 5 "" H 4800 1600 50  0001 L CNN "Height"
-F 6 "7981195P" H 4800 1500 50  0001 L CNN "RS Part Number"
-F 7 "Texas Instruments" H 4800 1400 50  0001 L CNN "Manufacturer_Name"
-F 8 "LMZ14202TZE-ADJ/NOPB" H 4800 1300 50  0001 L CNN "Manufacturer_Part_Number"
+F 5 "7981195P" H 4800 1500 50  0001 L CNN "RS Part Number"
+F 6 "Texas Instruments" H 4800 1400 50  0001 L CNN "Manufacturer_Name"
+F 7 "LMZ14202TZE-ADJ/NOPB" H 4800 1300 50  0001 L CNN "Manufacturer_Part_Number"
 	1    3750 1800
 	1    0    0    -1
@@
 P 2700 1400
 F 0 "R29" H 2770 1446 50  0000 L CNN
-F 1 "68.1k" H 2770 1355 50  0000 L CNN
-F 2 "Resistors_SMD:R_0603" V 2630 1400 50  0001 C CNN
+F 1 "68k" H 2770 1355 50  0000 L CNN
+F 2 "Resistor_SMD:R_0603_1608Metric_Pad1.05x0.95mm_HandSolder" V 2630 1400 50  0001 C CNN
 F 3 "~" H 2700 1400 50  0001 C CNN
 	1    2700 1400
@@
 F 0 "R30" H 2770 1996 50  0000 L CNN
 F 1 "11.8k" H 2770 1905 50  0000 L CNN
-F 2 "Resistors_SMD:R_0603" V 2630 1950 50  0001 C CNN
+F 2 "Resistor_SMD:R_0603_1608Metric_Pad1.05x0.95mm_HandSolder" V 2630 1950 50  0001 C CNN
 F 3 "~" H 2700 1950 50  0001 C CNN
 	1    2700 1950
@@
 F 0 "R31" H 3270 1446 50  0000 L CNN
 F 1 "100k" H 3270 1355 50  0000 L CNN
-F 2 "Resistors_SMD:R_0603" V 3130 1400 50  0001 C CNN
+F 2 "Resistor_SMD:R_0603_1608Metric_Pad1.05x0.95mm_HandSolder" V 3130 1400 50  0001 C CNN
 F 3 "~" H 3200 1400 50  0001 C CNN
 	1    3200 1400
@@
 F 0 "R34" H 6120 1946 50  0000 L CNN
 F 1 "5.62k" H 6120 1855 50  0000 L CNN
-F 2 "Resistors_SMD:R_0603" V 5980 1900 50  0001 C CNN
+F 2 "Resistor_SMD:R_0603_1608Metric_Pad1.05x0.95mm_HandSolder" V 5980 1900 50  0001 C CNN
 F 3 "~" H 6050 1900 50  0001 C CNN
 	1    6050 1900
@@
 F 0 "R32" H 5670 2096 50  0000 L CNN
 F 1 "1.07k" H 5670 2005 50  0000 L CNN
-F 2 "Resistors_SMD:R_0603" V 5530 2050 50  0001 C CNN
+F 2 "Resistor_SMD:R_0603_1608Metric_Pad1.05x0.95mm_HandSolder" V 5530 2050 50  0001 C CNN
 F 3 "~" H 5600 2050 50  0001 C CNN
 	1    5600 2050
@@
 F 0 "C21" V 5798 1350 50  0000 C CNN
 F 1 "22n" V 5889 1350 50  0000 C CNN
-F 2 "Capacitors_SMD:C_0805" H 6088 1200 50  0001 C CNN
+F 2 "Capacitor_SMD:C_0805_2012Metric_Pad1.15x1.40mm_HandSolder" H 6088 1200 50  0001 C CNN
 F 3 "~" H 6050 1350 50  0001 C CNN
 	1    6050 1350
@@
 F 0 "C22" H 6565 2096 50  0000 L CNN
 F 1 "1u" H 6565 2005 50  0000 L CNN
-F 2 "Capacitors_SMD:C_0805" H 6488 1900 50  0001 C CNN
+F 2 "Capacitor_SMD:C_0805_2012Metric_Pad1.15x1.40mm_HandSolder" H 6488 1900 50  0001 C CNN
 F 3 "~" H 6450 2050 50  0001 C CNN
 	1    6450 2050
@@
 F 0 "C23" H 7015 2096 50  0000 L CNN
 F 1 "100u" H 7015 2005 50  0000 L CNN
-F 2 "Capacitors_SMD:C_1210" H 6938 1900 50  0001 C CNN
+F 2 "Capacitor_SMD:C_1206_3216Metric_Pad1.42x1.75mm_HandSolder" H 6938 1900 50  0001 C CNN
 F 3 "~" H 6900 2050 50  0001 C CNN
 	1    6900 2050
@@
 F 0 "C6" H 2315 1696 50  0000 L CNN
 F 1 "10u" H 2315 1605 50  0000 L CNN
-F 2 "Capacitors_SMD:C_1206" H 2238 1500 50  0001 C CNN
+F 2 "Capacitor_SMD:C_1206_3216Metric_Pad1.42x1.75mm_HandSolder" H 2238 1500 50  0001 C CNN
 F 3 "~" H 2200 1650 50  0001 C CNN
 	1    2200 1650
@@
 F 0 "C5" H 1865 1696 50  0000 L CNN
 F 1 "1u" H 1865 1605 50  0000 L CNN
-F 2 "Capacitors_SMD:C_0805" H 1788 1500 50  0001 C CNN
+F 2 "Capacitor_SMD:C_0805_2012Metric_Pad1.15x1.40mm_HandSolder" H 1788 1500 50  0001 C CNN
 F 3 "~" H 1750 1650 50  0001 C CNN
 	1    1750 1650
@@
 F 0 "C19" H 5215 1446 50  0000 L CNN
 F 1 "22n" H 5215 1355 50  0000 L CNN
-F 2 "Capacitors_SMD:C_0805" H 5138 1250 50  0001 C CNN
+F 2 "Capacitor_SMD:C_0805_2012Metric_Pad1.15x1.40mm_HandSolder" H 5138 1250 50  0001 C CNN
 F 3 "~" H 5100 1400 50  0001 C CNN
 	1    5100 1400
@@
 F 0 "D1" H 1350 1034 50  0000 C CNN
 F 1 "D" H 1350 1125 50  0000 C CNN
-F 2 "Diodes_SMD:D_SOD-123" H 1350 1250 50  0001 C CNN
+F 2 "Diode_SMD:D_SOD-123" H 1350 1250 50  0001 C CNN
 F 3 "~" H 1350 1250 50  0001 C CNN
 	1    1350 1250
@@
 F 0 "C15" H 2815 3746 50  0000 L CNN
 F 1 "1u" H 2815 3655 50  0000 L CNN
-F 2 "Capacitors_SMD:C_0805" H 2738 3550 50  0001 C CNN
+F 2 "Capacitor_SMD:C_0805_2012Metric_Pad1.15x1.40mm_HandSolder" H 2738 3550 50  0001 C CNN
 F 3 "~" H 2700 3700 50  0001 C CNN
 	1    2700 3700
@@
 +5v
 Wire Wire Line
-	6900 1900 7250 1900
+	6900 1900 7050 1900
 Wire Wire Line
 	6450 1900 6900 1900
@@
 F 0 "R35" H 7470 2096 50  0000 L CNN
 F 1 "1.2k" H 7470 2005 50  0000 L CNN
-F 2 "Resistors_SMD:R_0603" V 7330 2050 50  0001 C CNN
+F 2 "Resistor_SMD:R_0603_1608Metric_Pad1.05x0.95mm_HandSolder" V 7330 2050 50  0001 C CNN
 F 3 "~" H 7400 2050 50  0001 C CNN
 	1    7400 2050
@@
 F 0 "D3" V 7438 2233 50  0000 R CNN
 F 1 "LED" V 7347 2233 50  0000 R CNN
-F 2 "Diodes_SMD:D_0805" H 7400 2350 50  0001 C CNN
+F 2 "LED_SMD:LED_0805_2012Metric_Pad1.15x1.40mm_HandSolder" H 7400 2350 50  0001 C CNN
 F 3 "~" H 7400 2350 50  0001 C CNN
 	1    7400 2350
@@
 F 0 "R33" H 5470 3746 50  0000 L CNN
 F 1 "1.2k" H 5470 3655 50  0000 L CNN
-F 2 "Resistors_SMD:R_0603" V 5330 3700 50  0001 C CNN
+F 2 "Resistor_SMD:R_0603_1608Metric_Pad1.05x0.95mm_HandSolder" V 5330 3700 50  0001 C CNN
 F 3 "~" H 5400 3700 50  0001 C CNN
 	1    5400 3700
@@
 F 0 "D2" V 5438 3883 50  0000 R CNN
 F 1 "LED" V 5347 3883 50  0000 R CNN
-F 2 "Diodes_SMD:D_0805" H 5400 4000 50  0001 C CNN
+F 2 "LED_SMD:LED_0805_2012Metric_Pad1.15x1.40mm_HandSolder" H 5400 4000 50  0001 C CNN
 F 3 "~" H 5400 4000 50  0001 C CNN
 	1    5400 4000
@@
 F 0 "U3" H 3550 3792 50  0000 C CNN
 F 1 "LM1117-3.3" H 3550 3701 50  0000 C CNN
-F 2 "TO_SOT_Packages_SMD:SOT-223" H 3550 3550 50  0001 C CNN
+F 2 "Package_TO_SOT_SMD:SOT-223" H 3550 3550 50  0001 C CNN
 F 3 "http://www.ti.com/lit/ds/symlink/lm1117.pdf" H 3550 3550 50  0001 C CNN
 F 4 "LM1117MP-3.3/NOPB" H 0   0   50  0001 C CNN "Manufacturer_Part_Number"
@@
 F 0 "C33" H 4215 3846 50  0000 L CNN
 F 1 "100n" H 4215 3755 50  0000 L CNN
-F 2 "Capacitors_SMD:C_0805" H 4138 3650 50  0001 C CNN
+F 2 "Capacitor_SMD:C_0805_2012Metric_Pad1.15x1.40mm_HandSolder" H 4138 3650 50  0001 C CNN
 F 3 "~" H 4100 3800 50  0001 C CNN
 	1    4100 3800
@@
 F 0 "C34" H 4665 3846 50  0000 L CNN
 F 1 "10u" H 4665 3755 50  0000 L CNN
-F 2 "Capacitors_SMD:C_0805" H 4588 3650 50  0001 C CNN
+F 2 "Capacitor_SMD:C_1206_3216Metric_Pad1.42x1.75mm_HandSolder" H 4588 3650 50  0001 C CNN
 F 3 "~" H 4550 3800 50  0001 C CNN
 	1    4550 3800
 	1    0    0    -1
 $EndComp
+$Comp
+L power:+5V #PWR0134
+U 1 1 5CB3C901
+P 7050 1900
+F 0 "#PWR0134" H 7050 1750 50  0001 C CNN
+F 1 "+5V" H 7065 2073 50  0000 C CNN
+F 2 "" H 7050 1900 50  0001 C CNN
+F 3 "" H 7050 1900 50  0001 C CNN
+	1    7050 1900
+	1    0    0    -1
+$EndComp
+Connection ~ 7050 1900
+Wire Wire Line
+	7050 1900 7250 1900
 $EndSCHEMATC
